File: OpAmpBasics/Ep004-DiffAmp/demos/demos.kicad_sch (KiCad schematic)
At the start: 44 parts, among them J1 AudioJack3, J2 AudioJack3, J3 Conn_01x04_Socket, J4 Conn_01x04_Socket, J5 Conn_01x02_Socket, J6 Conn_01x02_Socket, J7 Conn_01x02_Socket, J8 Conn_01x02_Socket, U1 LMC6482, U2 TL072

Commit message: op-amp basics episode 4 - correct error in schematic where the ring connector of J1 is left floating while the tip connects to both channels of the output. Thanks to YouTube user @shean4 for catching the mistake.
Connections:
- net at J1.T, R4.1, R6.1: no longer R7.1
- net at J1.R, R2.1: now also R7.1
