File: Transistor101/Ep014-017_DiffPairs/LongTailedPair5/LongTailedPair5.kicad_sch (KiCad schematic)
At the start: 17 parts, among them J1 AWG channel 1, J2 AWG channel 2, J3 Output to oscilloscope, Q1 DMMT5551, Q2 DMMT5551, T1 SEE NOTES

Commit message: Transistor 101 - episodes 16-18
Parts:
- removed J2: AWG channel 2, symbol Connector:Conn_01x02_Socket
- removed R1: 100R, symbol Device:R_Small_US
- removed R2, R3: 300R, symbol Device:R_Small_US
- removed T1: SEE NOTES, symbol Device:Transformer_1P_SS
- added C5, C6: 100n, symbol Device:C_Small
- added C7: SEE BELOW, symbol Device:C_Small
- added Q3, Q5: 2N4403, symbol Device:Q_PNP_EBC
- added Q4: 2N4401, symbol Device:Q_NPN_EBC
- added R8: 300R, symbol Device:R_Small_US
- added R9: 12k, symbol Device:R_Small_US
- R5: value 24k -> 3k3
Connections:
- net V_{+} is gone; now on an unnamed net: Q1.2 (B2)
- net +12V: now also C5.1, Q4.3 (C), R8.1
- net -12V: now also C6.2, Q5.3 (C), R9.2
- net Earth: now also C5.2, C6.1
- net at Q1.5 (E1): now also Q1.4 (E2), Q2.3 (C2)
- net at Q1.3 (C2), R5.2: now also C7.1, Q3.2 (B); no longer J3.1 (Pin_1)
- net V_{-}: no longer names the net of Q1.1 (B1)
- net V_{-}: now also J3.1 (Pin_1), Q4.1 (E), Q5.1 (E)
- new net: C7.2, Q3.3 (C), Q4.2 (B), Q5.2 (B), R9.1
- new net: Q3.1 (E), R8.2
Other:
- note added: "FOLLOWER STAGE"
- note added: "GAIN STAGE"
- note added: "INPUT SIGNAL"
- note added: "OSCILLOSCOPE"
- note added: "Place C3, C4 as close to Q1 as possible. Place C5, C6 as close to Q4 and Q5 as possible."
- note added: "Select C7 as needed to eliminate spurious high-frequency oscillation when amplifier is configured for unity gain. 100 pF is suggested as a starting value. Increase if oscillations are not cured; cautiously decrease if oscillations are cured, to see what speed is achievable. 33 pF worked in my setup (somewhat surprisingly - I expected to need more)"
- note added: "This circuit can be breadboarded starting with the circuit from episode 17, replacing the feedback divider with a simple wire. 1. Make the modification, observe unity gain but likely high-frequency oscillation. 2. Attenpt to cure the oscillation by adding compensation capacitor C7."
- note removed: "COMMON MODE SIGNAL"
- note removed: "DIFFERENTIAL MODE SIGNAL"
- note removed: "Place C3, C4 as close to Q1 as possible."
- note removed: "T1 is a small 120V:6.3VCT power transformer Triad Magnetics F-14X or similar. Suitable transformers can often be scavenged from discarded equipment with linear power supplies."
- note removed: "TEST RIG"
- note removed: "Test rig allows testing the pair's response to common mode and differential signals, together or separately. When applying the common mode signal by itself, it is advantageous to short pins 1 and 2 of Q1 with a short jumper to avoid picking up spurious differences."
- note removed: "This circuit can be breadboarded starting with the circuit from episode 14, removing R4 and replacing it with the current source. All other subcircuits are unchanged between the two episodes. Test first with R2 and R3 in place. Then remove R2 and R3 and replace with short circuits. Observe that the gain is improved, the CMRR is unchanged, the circuit remains thermally stable, but large signals su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"
- moved on the sheet: C1, C2, C3, C4, J1, J3, Q1A, Q1B, Q2A, Q2B, R4, R5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

Commit message: Correct pinout of DMMT5401
Parts:
- Q1, Q2: footprint (none) -> Package_TO_SOT_SMD:SOT-363_SC-70-6; symbol Kevin-Transistors:Q_Dual_NPN_NPN_B1B2C2E2E1C1 -> Kevin-Transistors:DMMT5551
Connections:
- net +12V: now also Q1.1 (C1); no longer Q1.6 (C1)
- net at J3.1 (Pin_1), Q4.1 (E), Q5.1 (E): now also Q1.2 (B1); no longer Q1.1 (B1)
- net at R6.1: now also Q2.6 (E1); no longer Q2.5 (E1)
- net at J1.1 (Pin_1): now also Q1.3 (B2); no longer Q1.2 (B2)
- net at Q2.1 (C1), R4.2: now also Q2.2 (B1), Q2.3 (B2); no longer Q2.2 (B2), Q2.6 (C1)
- net at C7.1, Q3.2 (B), R5.2: now also Q1.4 (C2); no longer Q1.3 (C2)
- net at Q2.4 (C2): now also Q1.5 (E2), Q1.6 (E1); no longer R7.1
- new net: Q2.5 (E2), R7.1
Changed lines of the file:
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@@
   (title_block
     (title "Long-tailed pair: the basic circuit")
-    (date "2025-02-08")
-    (rev "A")
+    (date "2026-05-13")
+    (rev "B")
     (company "Kludges from Kevin's Cave")
     (comment 1 "The differential pair becomes an op-amp")
@@
     )
   )
-  (symbol (lib_id "Kevin-Transistors:Q_Dual_NPN_NPN_B1B2C2E2E1C1") (at 102.87 119.38 0) (mirror y) (unit 1)
+  (symbol (lib_id "Kevin-Transistors:DMMT5551") (at 102.87 119.38 0) (mirror y) (unit 1)
     (in_bom yes) (on_board yes) (dnp no)
     (property "Reference" "Q2" (at 96.52 118.11 0)
@@
       (effects (font (size 1.27 1.27)) (justify left))
     )
-    (property "Footprint" "" (at 97.79 116.84 0)
-      (effects (font (size 1.27 1.27)) hide)
-    )
-    (property "Datasheet" "~" (at 102.87 119.38 0)
+    (property "Footprint" "Package_TO_SOT_SMD:SOT-363_SC-70-6" (at 97.79 116.84 0)
+      (effects (font (size 1.27 1.27)) hide)
+    )
+    (property "Datasheet" "https://www.diodes.com/assets/Datasheets/ds30436.pdf" (at 102.87 119.38 0)
       (effects (font (size 1.27 1.27)) hide)
     )
@@
     )
   )
-  (symbol (lib_id "Kevin-Transistors:Q_Dual_NPN_NPN_B1B2C2E2E1C1") (at 134.62 74.93 0) (mirror y) (unit 2)
+  (symbol (lib_id "Kevin-Transistors:DMMT5551") (at 134.62 74.93 0) (mirror y) (unit 2)
     (in_bom yes) (on_board yes) (dnp no)
     (property "Reference" "Q1" (at 139.7 71.12 0)
@@
       (effects (font (size 1.27 1.27)) (justify left) hide)
     )
-    (property "Footprint" "" (at 129.54 72.39 0)
-      (effects (font (size 1.27 1.27)) hide)
-    )
-    (property "Datasheet" "~" (at 134.62 74.93 0)
+    (property "Footprint" "Package_TO_SOT_SMD:SOT-363_SC-70-6" (at 129.54 72.39 0)
+      (effects (font (size 1.27 1.27)) hide)
+    )
+    (property "Datasheet" "https://www.diodes.com/assets/Datasheets/ds30436.pdf" (at 134.62 74.93 0)
       (effects (font (size 1.27 1.27)) hide)
     )
@@
     )
   )
-  (symbol (lib_id "Kevin-Transistors:Q_Dual_NPN_NPN_B1B2C2E2E1C1") (at 118.11 119.38 0) (unit 2)
+  (symbol (lib_id "Kevin-Transistors:DMMT5551") (at 118.11 119.38 0) (unit 2)
     (in_bom yes) (on_board yes) (dnp no)
     (property "Reference" "Q2" (at 124.46 116.84 0)
@@
       (effects (font (size 1.27 1.27)) (justify left) hide)
     )
-    (property "Footprint" "" (at 123.19 116.84 0)
-      (effects (font (size 1.27 1.27)) hide)
-    )
-    (property "Datasheet" "~" (at 118.11 119.38 0)
+    (property "Footprint" "Package_TO_SOT_SMD:SOT-363_SC-70-6" (at 123.19 116.84 0)
+      (effects (font (size 1.27 1.27)) hide)
+    )
+    (property "Datasheet" "https://www.diodes.com/assets/Datasheets/ds30436.pdf" (at 118.11 119.38 0)
       (effects (font (size 1.27 1.27)) hide)
     )
@@
     )
   )
-  (symbol (lib_id "Kevin-Transistors:Q_Dual_NPN_NPN_B1B2C2E2E1C1") (at 106.68 74.93 0) (unit 1)
+  (symbol (lib_id "Kevin-Transistors:DMMT5551") (at 106.68 74.93 0) (unit 1)
     (in_bom yes) (on_board yes) (dnp no)
     (property "Reference" "Q1" (at 102.87 71.12 0)
@@
       (effects (font (size 1.27 1.27)) (justify left))
     )
-    (property "Footprint" "" (at 111.76 72.39 0)
-      (effects (font (size 1.27 1.27)) hide)
-    )
-    (property "Datasheet" "~" (at 106.68 74.93 0)
-      (effects (font (size 1.27 1.27)) hide)
-    )
+    (property "Footprint" "Package_TO_SOT_SMD:SOT-363_SC-70-6" (at 111.76 72.39 0)
+      (effects (font (size 1.27 1.27)) hide)
+    )
+    (property "Datasheet" "https://www.diodes.com/assets/Datasheets/ds30436.pdf" (at 106.68 74.93 0)
+      (effects (font (size 1.27 1.27)) hide)
+    )
